File: Adapter-VCNL4200.kicad_pcb (KiCad board)
At the start: 2 copper layers, 13.5 x 13 mm, 9 parts, among them J1 Conn_01x04, J2 Conn_01x04, U1 VCNL4200

Commit message: Created gerbers
Parts:
- moved R2 2.00 mm to (156.0, 129.0)
- moved R3 2.00 mm to (156.0, 131.0)
Routing:
- net VCC: track 0.00 -> 16.6 mm
- net /INT: track 0.00 -> 9.26 mm
- net /SDAT: track 0.00 -> 8.69 mm
- net /SCLK: track 0.00 -> 8.39 mm
- net /LED-: track 0.00 -> 8.14 mm
- net GND: track 0.00 -> 7.67 mm
- net /LED_CATHODE: track 0.00 -> 3.73 mm
- net /LED+: track 0.00 -> 3.64 mm
- added copper zone on B.Cu, net GND
Other:
- net class Default: trace_width 0.25 -> 0.2
- rule via_min_size: 0.4 -> 0.6
